Commit message: update-2025.10.12

File: tugbot_gazebo_my/urdf/tugbot.urdf (robot description, URDF)
Before this commit: robot tugbot, 11 links, 10 joints
Links:
- removed link tugbot/scan_back/scan_back
- removed link tugbot/scan_front/scan_front
- removed link tugbot/scan_omni/scan_omni
- added link scan_back
- added link scan_front
- added link scan_omni; visual cylinder length=0.0015 radius=0.06; visual cylinder length=0.09 radius=0.005
Joints:
- joint scan_back_joint: child tugbot/scan_back/scan_back -> scan_back
- joint scan_front_joint: child tugbot/scan_front/scan_front -> scan_front
- joint scan_omni_joint: child tugbot/scan_omni/scan_omni -> scan_omni

Commit message: update-2025.10.12-2

File: tugbot_gazebo_my/urdf/tugbot.urdf (robot description, URDF)
Before this commit: robot tugbot, 11 links, 10 joints
Links:
- link base_link: geometry visual mesh filename=package://tugbot_gazebo_my/models/meshes/base/movai_logo.dae; visual mesh filename=package://tugbot_gazebo_my/models/meshes/base/tugbot_simp.d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
- link scan_omni: geometry visual cylinder length=0.0015 radius=0.06; visual cylinder length=0.09 radius=0.005
- link wheel_left: geometry collision cylinder length=0.05 radius=0.195; visual mesh filename=package://tugbot_gazebo_my/models/meshes/wheel/wheel.dae
- link wheel_right: geometry collision cylinder length=0.05 radius=0.195; visual mesh filename=package://tugbot_gazebo_my/models/meshes/wheel/wheel.dae

Commit message: update-2025.10.14

File: tugbot_gazebo_my/urdf/tugbot.urdf (robot description, URDF)
Before this commit: robot tugbot, 11 links, 10 joints
Links:
- removed link tugbot/camera_back
- removed link tugbot/camera_front
- added link camera_back
- added link camera_front
- added link camera_front/color
- added link camera_front/depth
Joints:
- added joint camera_front_color_joint: type fixed, parent camera_front, child camera_front/color, origin xyz=0 0 0 rpy=0 0 0
- added joint camera_front_depth_joint: type fixed, parent camera_front, child camera_front/depth, origin xyz=0 0 0 rpy=0 0 0
- joint camera_back_joint: child tugbot/camera_back -> camera_back
- joint camera_front_joint: child tugbot/camera_front -> camera_front

Commit message: update-2025.10.16

File: tugbot_gazebo_my/urdf/tugbot.urdf (robot description, URDF)
Before this commit: robot tugbot, 13 links, 12 joints
Links:
- removed link camera_back
- removed link camera_front
- removed link camera_front/color
- removed link camera_front/depth
- added link camera_back_link
- added link camera_front/color_frame
- added link camera_front/color_optical_frame
- added link camera_front/depth_frame
- added link camera_front/depth_optical_frame
- added link camera_front_link
Joints:
- added joint camera_front_color_optical_joint: type fixed, parent camera_front_link, child camera_front/color_optical_frame, origin xyz=0 0.032500000000000001 0.012500000000000001 rpy=-1.5707963267948966 0 -1.5707963267948966
- added joint camera_front_depth_optical_joint: type fixed, parent camera_front_link, child camera_front/depth_optical_frame, origin xyz=0 0.017500000000000002 0.012500000000000001 rpy=-1.5707963267948966 0 -1.5707963267948966
- joint camera_back_joint: child camera_back -> camera_back_link
- joint camera_front_color_joint: child camera_front/color -> camera_front/color_frame; origin xyz=0 0 0 rpy=0 0 0 -> xyz=0 0.032500000000000001 0.012500000000000001 rpy=0 0 0; parent camera_front -> camera_front_link
- joint camera_front_depth_joint: child camera_front/depth -> camera_front/depth_frame; origin xyz=0 0 0 rpy=0 0 0 -> xyz=0 0.017500000000000002 0.012500000000000001 rpy=0 0 0; parent camera_front -> camera_front_link
- joint camera_front_joint: child camera_front -> camera_front_link; origin xyz=0.0553 0 0.4323 rpy=0 0 0 -> xyz=0.0553 0 0.275 rpy=0 0.017453292519943295 0

Commit message: update-2025.10.24

File: tugbot_gazebo_my/urdf/tugbot.urdf (robot description, URDF)
Before this commit: robot tugbot, 15 links, 14 joints
Joints:
- joint camera_front_color_joint: origin xyz=0 0.032500000000000001 0.012500000000000001 rpy=0 0 0 -> xyz=0 0 0 rpy=0 0 0
- joint camera_front_color_optical_joint: origin xyz=0 0.032500000000000001 0.012500000000000001 rpy=-1.5707963267948966 0 -1.5707963267948966 -> xyz=0 0 0 rpy=-1.5707963267948966 0 -1.5707963267948966; parent camera_front_link -> camera_front/color_frame
- joint camera_front_depth_joint: origin xyz=0 0.017500000000000002 0.012500000000000001 rpy=0 0 0 -> xyz=0 0.0175 0.0125 rpy=0 0 0
- joint camera_front_depth_optical_joint: origin xyz=0 0.017500000000000002 0.012500000000000001 rpy=-1.5707963267948966 0 -1.5707963267948966 -> xyz=0 0 0 rpy=-1.5707963267948966 0 -1.5707963267948966; parent camera_front_link -> camera_front/depth_frame
- joint camera_front_joint: origin xyz=0.0553 0 0.275 rpy=0 0.017453292519943295 0 -> xyz=0.0553 0 0.4323 rpy=0 0 0
